Commit message: Rename package and add meshes for some objects and features
* Rename package to motoman_ma2010_d500_waam_support
* Add meshes for manipulator riser, floor slab and substrate plate

File: urdf/ma2010_d500.xacro (robot description, xacro)
@@ -5,10 +5,46 @@
       <color rgba="0.12941 0.14902 0.74902 1" />
   </material>
-	<xacro:include filename="$(find motoman_ma2010_motopos_d500_support)/urdf/ma2010_d500_macro.xacro" />
+  <material name="grey">
+      <color rgba="0.5 0.5 0.5 1" />
+  </material>
+  <material name="black">
+      <color rgba="0 0 0 1" />
+  </material>
+	<xacro:include filename="$(find motoman_ma2010_d500_waam_support)/urdf/ma2010_d500_macro.xacro" />
 	<xacro:ma2010_d500 prefix=""/>
   <!-- ROS base_link to Robot Manufacturer World Coordinates transform -->
-	<link name="world" />
+  <!-- TODO create a separate xacro:macro for this -->
+	<link name="world" >
+    <!-- manipulator riser -->
+    <visual>
+      <origin xyz="-0.2725 -0.2725 0"/>
+      <geometry>
+        <mesh filename="package://motoman_ma2010_d500_waam_support/meshes/15067-2_460mm_m.stl"/>
+      </geometry>
+      <material name="grey"/>
+    </visual>
+    <collision>
+      <origin xyz="-0.2725 -0.2725 0"/>
+      <geometry>
+        <mesh filename="package://motoman_ma2010_d500_waam_support/meshes/15067-2_460mm_m.stl"/>
+      </geometry>
+    </collision>
+    <!-- floor slab -->
+    <visual>
+      <origin xyz="-0.85 -1.25 0" rpy="1.58 0 1.58"/>
+      <geometry>
+        <mesh filename="package://motoman_ma2010_d500_waam_support/meshes/floor_slab_m.stl"/>
+      </geometry>
+      <material name="grey"/>
+    </visual>
+    <collision>
+      <origin xyz="-0.85 -1.25 0" rpy="1.58 0 1.58"/>
+      <geometry>
+        <mesh filename="package://motoman_ma2010_d500_waam_support/meshes/floor_slab_m.stl"/>
+      </geometry>
+    </collision>
+  </link>
   <joint name="d500_base_link-world" type="fixed">
-    <origin xyz="1.25 0 0" rpy="0 0 -1.58"/>
+    <origin xyz="1.35 0 0" rpy="0 0 -1.58"/>
     <parent link="world"/>
     <child link="d500_base_link"/>
@@ -19,3 +55,24 @@
     <child link="ma2010_base_link"/>
   </joint>
+  <!-- Substrate plate on the positioner -->
+  <link name="d500_sub_plate">
+    <visual>
+      <origin xyz="-0.25 -0.25 0"/>
+      <geometry>
+        <mesh filename="package://motoman_ma2010_d500_waam_support/meshes/substrate_plate_m.stl"/>
+      </geometry>
+      <material name="grey"/>
+    </visual>
+    <collision>
+      <origin xyz="-0.25 -0.25 0"/>
+      <geometry>
+        <mesh filename="package://motoman_ma2010_d500_waam_support/meshes/substrate_plate_m.stl"/>
+      </geometry>
+    </collision>
+  </link>
+  <joint name="d500_tool0-d500_sub_plate" type="fixed">
+    <parent link="d500_tool0" />
+    <child link="d500_sub_plate" />
+    <origin xyz="0 0 0" rpy="0 0 0"/>
+  </joint>
 </robot>

Commit message: Add torch mesh and incorporate into the urdf model

File: urdf/ma2010_d500.xacro (robot description, xacro)
@@ -32,5 +32,5 @@
     <!-- floor slab -->
     <visual>
-      <origin xyz="-0.85 -1.25 0" rpy="1.58 0 1.58"/>
+      <origin xyz="-0.85 -1.25 0" rpy="${pi/2} 0 ${pi/2}"/>
       <geometry>
         <mesh filename="package://motoman_ma2010_d500_waam_support/meshes/floor_slab_m.stl"/>
@@ -39,5 +39,5 @@
     </visual>
     <collision>
-      <origin xyz="-0.85 -1.25 0" rpy="1.58 0 1.58"/>
+      <origin xyz="-0.85 -1.35 0" rpy="${pi/2} 0 ${pi/2}"/>
       <geometry>
         <mesh filename="package://motoman_ma2010_d500_waam_support/meshes/floor_slab_m.stl"/>
@@ -46,5 +46,5 @@
   </link>
   <joint name="d500_base_link-world" type="fixed">
-    <origin xyz="1.35 0 0" rpy="0 0 -1.58"/>
+    <origin xyz="1.35 0 0" rpy="0 0 -${pi/2}"/>
     <parent link="world"/>
     <child link="d500_base_link"/>
@@ -58,5 +58,5 @@
   <link name="d500_sub_plate">
     <visual>
-      <origin xyz="-0.25 -0.25 0"/>
+      <origin xyz="-0.25 -0.25 -0.01"/>
       <geometry>
         <mesh filename="package://motoman_ma2010_d500_waam_support/meshes/substrate_plate_m.stl"/>
@@ -74,5 +74,32 @@
     <parent link="d500_tool0" />
     <child link="d500_sub_plate" />
-    <origin xyz="0 0 0" rpy="0 0 0"/>
+    <origin xyz="0 0 0.01" rpy="0 0 ${pi/2}"/>
+  </joint>
+  <!-- Tool (torch) -->
+  <link name="ma2010_tool_tip">
+    <visual>
+      <origin xyz="0 0.035 0.195" rpy="${pi/2} ${pi} 0"/>
+      <geometry>
+        <mesh filename="package://motoman_ma2010_d500_waam_support/meshes/ra_5000_22g.stl"/>
+      </geometry>
+      <material name="grey"/>
+    </visual>
+    <collision>
+      <origin xyz="0 0.035 0.195" rpy="${pi/2} ${pi} 0"/>
+      <geometry>
+        <mesh filename="package://motoman_ma2010_d500_waam_support/meshes/ra_5000_22g.stl"/>
+      </geometry>
+    </collision>
+  </link>
+  <joint name="ma2010_tool0-ma2010_tool_tip" type="fixed">
+    <parent link="ma2010_tool0" />
+    <child link="ma2010_tool_tip" />
+    <origin xyz="0.4299 0 0" rpy="0 0 0"/>
+  </joint>
+  <link name="ma2010_tool_tip_ang" />
+  <joint name="ma2010_tool0-ma2010_tool_tip_ang" type="fixed">
+    <parent link="ma2010_tool_tip" />
+    <child link="ma2010_tool_tip_ang" />
+    <origin xyz="0 0 0" rpy="0 -0.91 0"/>
   </joint>
 </robot>

Commit message: Fix floor slab positioning

File: urdf/ma2010_d500.xacro (robot description, xacro)
@@ -39,5 +39,5 @@
     </visual>
     <collision>
-      <origin xyz="-0.85 -1.35 0" rpy="${pi/2} 0 ${pi/2}"/>
+      <origin xyz="-0.85 -1.25 0" rpy="${pi/2} 0 ${pi/2}"/>
       <geometry>
         <mesh filename="package://motoman_ma2010_d500_waam_support/meshes/floor_slab_m.stl"/>

Commit message: Add positioner base plate

File: urdf/ma2010_d500.xacro (robot description, xacro)
@@ -44,7 +44,21 @@
       </geometry>
     </collision>
+    <!-- positioner base plate -->
+    <visual>
+      <origin xyz="0.85 -0.4 0" rpy="0 0 0"/>
+      <geometry>
+        <mesh filename="package://motoman_ma2010_d500_waam_support/meshes/base_plate_positioner_m.stl"/>
+      </geometry>
+      <material name="grey"/>
+    </visual>
+    <collision>
+      <origin xyz="0.85 -0.4 0" rpy="0 0 0"/>
+      <geometry>
+        <mesh filename="package://motoman_ma2010_d500_waam_support/meshes/base_plate_positioner_m.stl"/>
+      </geometry>
+    </collision>
   </link>
   <joint name="d500_base_link-world" type="fixed">
-    <origin xyz="1.35 0 0" rpy="0 0 -${pi/2}"/>
+    <origin xyz="1.35 0 0.032" rpy="0 0 -${pi/2}"/>
     <parent link="world"/>
     <child link="d500_base_link"/>

Commit message: Add manipulator tcp (torch tip + 15 mm stick-out)

File: urdf/ma2010_d500.xacro (robot description, xacro)
@@ -117,3 +117,9 @@
     <origin xyz="0 0 0" rpy="0 -0.91 0"/>
   </joint>
+  <link name="ma2010_tcp" />
+  <joint name="ma2010_tool_tip_ang-ma2010_tcp" type="fixed">
+    <parent link="ma2010_tool_tip_ang" />
+    <child link="ma2010_tcp" />
+    <origin xyz="0 0 -0.015" rpy="0 0 0"/>
+  </joint>
 </robot>

Commit message: Add correct torch model and add temporary substrate plate

File: urdf/ma2010_d500.xacro (robot description, xacro)
@@ -60,5 +60,5 @@
   </link>
   <joint name="d500_base_link-world" type="fixed">
-    <origin xyz="1.35 0 0.032" rpy="0 0 -${pi/2}"/>
+    <origin xyz="1.365256 0 0.032" rpy="0 0 -${pi/2}"/>
     <parent link="world"/>
     <child link="d500_base_link"/>
@@ -72,14 +72,14 @@
   <link name="d500_sub_plate">
     <visual>
-      <origin xyz="-0.25 -0.25 -0.01"/>
+      <origin xyz="-0.25 -0.25 -0.049"/>
       <geometry>
-        <mesh filename="package://motoman_ma2010_d500_waam_support/meshes/substrate_plate_m.stl"/>
+        <mesh filename="package://motoman_ma2010_d500_waam_support/meshes/substrate_plate_temp_m.stl"/>
       </geometry>
       <material name="grey"/>
     </visual>
     <collision>
-      <origin xyz="-0.25 -0.25 0"/>
+      <origin xyz="-0.25 -0.25 -0.049"/>
       <geometry>
-        <mesh filename="package://motoman_ma2010_d500_waam_support/meshes/substrate_plate_m.stl"/>
+        <mesh filename="package://motoman_ma2010_d500_waam_support/meshes/substrate_plate_temp_m.stl"/>
       </geometry>
     </collision>
@@ -88,26 +88,33 @@
     <parent link="d500_tool0" />
     <child link="d500_sub_plate" />
-    <origin xyz="0 0 0.01" rpy="0 0 ${pi/2}"/>
+    <origin xyz="0 0 0.049" rpy="0 0 ${pi/2}"/>
   </joint>
   <!-- Tool (torch) -->
-  <link name="ma2010_tool_tip">
+  <link name="ma2010_torch">
     <visual>
-      <origin xyz="0 0.035 0.195" rpy="${pi/2} ${pi} 0"/>
+      <!--<origin xyz="-0.100 0.042 -0.050" rpy="${pi/2} 0.38 0"/>-->
+      <origin xyz="0 0 0" rpy="0 0 0"/>
       <geometry>
-        <mesh filename="package://motoman_ma2010_d500_waam_support/meshes/ra_5000_22g.stl"/>
+        <mesh filename="package://motoman_ma2010_d500_waam_support/meshes/RA_5000_22g.stl"/>
       </geometry>
       <material name="grey"/>
     </visual>
     <collision>
-      <origin xyz="0 0.035 0.195" rpy="${pi/2} ${pi} 0"/>
+      <origin xyz="0 0 0" rpy="0 0 0"/>
       <geometry>
-        <mesh filename="package://motoman_ma2010_d500_waam_support/meshes/ra_5000_22g.stl"/>
+        <mesh filename="package://motoman_ma2010_d500_waam_support/meshes/RA_5000_22g.stl"/>
       </geometry>
     </collision>
   </link>
+  <joint name="ma2010_tool0-ma2010_torch" type="fixed">
+    <parent link="ma2010_tool0"/>
+    <child link="ma2010_torch"/>
+    <origin xyz="0 0 0" rpy="0 0 0"/>
+  </joint>
+  <link name="ma2010_tool_tip" />
   <joint name="ma2010_tool0-ma2010_tool_tip" type="fixed">
-    <parent link="ma2010_tool0" />
+    <parent link="ma2010_torch" />
     <child link="ma2010_tool_tip" />
-    <origin xyz="0.4299 0 0" rpy="0 0 0"/>
+    <origin xyz="0.4754 0 0" rpy="0 0 0"/>
   </joint>
   <link name="ma2010_tool_tip_ang" />

Commit message: Fix typo in STL file name

File: urdf/ma2010_d500.xacro (robot description, xacro)
@@ -96,5 +96,5 @@
       <origin xyz="0 0 0" rpy="0 0 0"/>
       <geometry>
-        <mesh filename="package://motoman_ma2010_d500_waam_support/meshes/RA_5000_22g.stl"/>
+        <mesh filename="package://motoman_ma2010_d500_waam_support/meshes/ra_5000_22g.stl"/>
       </geometry>
       <material name="grey"/>
@@ -103,5 +103,5 @@
       <origin xyz="0 0 0" rpy="0 0 0"/>
       <geometry>
-        <mesh filename="package://motoman_ma2010_d500_waam_support/meshes/RA_5000_22g.stl"/>
+        <mesh filename="package://motoman_ma2010_d500_waam_support/meshes/ra_5000_22g.stl"/>
       </geometry>
     </collision>

Commit message: Add fixed torch model, change TCP, fix "d500_sub_plate" frame & rename

File: urdf/ma2010_d500.xacro (robot description, xacro)
@@ -60,5 +60,6 @@
   </link>
   <joint name="d500_base_link-world" type="fixed">
-    <origin xyz="1.365256 0 0.032" rpy="0 0 -${pi/2}"/>
+    <!--<origin xyz="1.373 0.0 0.032" rpy="0 0 -${pi/2}"/>-->
+    <origin xyz="1.348 -0.0015 0.032" rpy="0 0 -${pi/2}"/>
     <parent link="world"/>
     <child link="d500_base_link"/>
@@ -70,23 +71,23 @@
   </joint>
   <!-- Substrate plate on the positioner -->
-  <link name="d500_sub_plate">
+  <link name="d500_fix_plate">
     <visual>
-      <origin xyz="-0.25 -0.25 -0.049"/>
+      <origin xyz="-0.25 -0.25 -0.063"/>
       <geometry>
-        <mesh filename="package://motoman_ma2010_d500_waam_support/meshes/substrate_plate_temp_m.stl"/>
+        <mesh filename="package://motoman_ma2010_d500_waam_support/meshes/fixture_plate_m.stl"/>
       </geometry>
       <material name="grey"/>
     </visual>
     <collision>
-      <origin xyz="-0.25 -0.25 -0.049"/>
+      <origin xyz="-0.25 -0.25 -0.063"/>
       <geometry>
-        <mesh filename="package://motoman_ma2010_d500_waam_support/meshes/substrate_plate_temp_m.stl"/>
+        <mesh filename="package://motoman_ma2010_d500_waam_support/meshes/fixture_plate_m.stl"/>
       </geometry>
     </collision>
   </link>
-  <joint name="d500_tool0-d500_sub_plate" type="fixed">
+  <joint name="d500_tool0-d500_fix_plate" type="fixed">
     <parent link="d500_tool0" />
-    <child link="d500_sub_plate" />
-    <origin xyz="0 0 0.049" rpy="0 0 ${pi/2}"/>
+    <child link="d500_fix_plate" />
+    <origin xyz="0 0 0.063" rpy="0 0 ${pi/2}"/>
   </joint>
   <!-- Tool (torch) -->
@@ -96,5 +97,5 @@
       <origin xyz="0 0 0" rpy="0 0 0"/>
       <geometry>
-        <mesh filename="package://motoman_ma2010_d500_waam_support/meshes/ra_5000_22g.stl"/>
+        <mesh filename="package://motoman_ma2010_d500_waam_support/meshes/RA_5000_22g_7.5degree_fix.STL"/>
       </geometry>
       <material name="grey"/>
@@ -103,5 +104,5 @@
       <origin xyz="0 0 0" rpy="0 0 0"/>
       <geometry>
-        <mesh filename="package://motoman_ma2010_d500_waam_support/meshes/ra_5000_22g.stl"/>
+        <mesh filename="package://motoman_ma2010_d500_waam_support/meshes/RA_5000_22g_7.5degree_fix.STL"/>
       </geometry>
     </collision>
@@ -116,17 +117,11 @@
     <parent link="ma2010_torch" />
     <child link="ma2010_tool_tip" />
-    <origin xyz="0.4754 0 0" rpy="0 0 0"/>
-  </joint>
-  <link name="ma2010_tool_tip_ang" />
-  <joint name="ma2010_tool0-ma2010_tool_tip_ang" type="fixed">
-    <parent link="ma2010_tool_tip" />
-    <child link="ma2010_tool_tip_ang" />
-    <origin xyz="0 0 0" rpy="0 -0.91 0"/>
+    <origin xyz="0.46374 0 -0.01518" rpy="0 0 0"/>
   </joint>
   <link name="ma2010_tcp" />
-  <joint name="ma2010_tool_tip_ang-ma2010_tcp" type="fixed">
-    <parent link="ma2010_tool_tip_ang" />
+  <joint name="ma2010_tool0-ma2010_tcp" type="fixed">
+    <parent link="ma2010_tool_tip" />
     <child link="ma2010_tcp" />
-    <origin xyz="0 0 -0.015" rpy="0 0 0"/>
+    <origin xyz="0 0 0" rpy="0 -0.777 0"/>
   </joint>
 </robot>
